Commit message: cleaned unwanted files

File: urdf/mobile_bot.urdf (robot description, URDF)
Before this commit: robot luqman_bot, 6 links, 5 joints
Links:
- added link left_finger, mass 0.01; collision box size=0.2 0.0025 0.02; visual box size=0.2 0.0025 0.02
- added link right_finger, mass 0.01; collision box size=0.2 0.0025 0.02; visual box size=0.2 0.0025 0.02
- link base_link: mass 1.0 -> 0.5; geometry collision box size=0.3 0.3 0.05; visual box size=0.3 0.3 0.05
- link front_caster_of_wheel: mass 0.1 -> 0.05; geometry collision box size=0.01 0.01 0.01; visual box size=0.01 0.01 0.01
- link front_wheel: mass 0.1 -> 0.05; geometry collision cylinder length=0.025 radius=0.0175; visual cylinder length=0.025 radius=0.0175
- link laser_scanner: geometry collision box size=0.05 0.05 0.05; visual box size=0.05 0.05 0.05
- link left_wheel: mass 0.1 -> 0.05; geometry collision cylinder length=0.025 radius=0.0175; visual cylinder length=0.025 radius=0.0175
- link right_wheel: mass 0.1 -> 0.05; geometry collision cylinder length=0.025 radius=0.0175; visual cylinder length=0.025 radius=0.0175
Joints:
- added joint left_finger_joint: type prismatic, parent base_link, child left_finger, origin xyz=0.22 0.13 0.01 rpy=0.0 0.0 0.0, axis 0 -1 0, limit lower=0.0 upper=0.05 effort=10 velocity=0.05
- added joint right_finger_joint: type prismatic, parent base_link, child right_finger, origin xyz=0.22 -0.13 0.01 rpy=0.0 0.0 0.0, axis 0 1 0, limit lower=0.0 upper=0.05 effort=10 velocity=0.05
- joint front_caster_of_wheel_joint: origin xyz=0.3 0.0 0.0 rpy=0.0 0.0 0.0 -> xyz=0.10 0.0 0.0 rpy=0.0 0.0 0.0
- joint front_wheel_joint: origin xyz=0.05 0.0 -0.05 rpy=-1.5708 0.0 0.0 -> xyz=0.025 0.0 -0.025 rpy=-1.5708 0.0 0.0
- joint left_wheel_joint: origin xyz=-0.2825 0.125 -0.05 rpy=-1.5708 0.0 0.0 -> xyz=-0.14125 0.0625 -0.025 rpy=-1.5708 0.0 0.0
- joint right_wheel_joint: origin xyz=-0.2825 -0.125 -0.05 rpy=-1.5708 0.0 0.0 -> xyz=-0.14125 -0.0625 -0.025 rpy=-1.5708 0.0 0.0

File: urdf/test.urdf (robot description, URDF)
Before this commit: robot my_robot, 6 links, 5 joints
Links:
- removed link base_footprint
Joints:
- removed joint base_link_to_base_footprint
- joint front_left_wheel_joint: origin xyz=0.25 0.15 -0.05 rpy=0 0 0 -> xyz=0.25 0.15 -0.05 rpy=1.57 0.0 0.0
- joint front_right_wheel_joint: origin xyz=0.25 -0.15 -0.05 rpy=0 0 0 -> xyz=0.25 -0.15 -0.05 rpy=1.57 0.0 0.0
- joint rear_left_wheel_joint: origin xyz=-0.25 0.15 -0.05 rpy=0 0 0 -> xyz=-0.25 0.15 -0.05 rpy=1.57 0.0 0.0
- joint rear_right_wheel_joint: origin xyz=-0.25 -0.15 -0.05 rpy=0 0 0 -> xyz=-0.25 -0.15 -0.05 rpy=1.57 0.0 0.0

File: urdf/test2.urdf (robot description, URDF)
Before this commit: robot my_robot, 6 links, 5 joints
Links:
- added link laser_scanner, mass 1e-5; collision box size=0.1 0.1 0.1; visual box size=0.1 0.1 0.1
- added link wheel_steering_link, mass 1e-5; collision box size=0.1 0.1 0.1; visual box size=0.1 0.1 0.1
Joints:
- added joint laser_scanner_joint: type fixed, parent base_link, child laser_scanner, origin xyz=0.0 0.0 0.08 rpy=0.0 0.0 0.0, axis 0.0 0.0 0.08
- added joint wheel_steering_joint: type revolute, parent base_link, child wheel_steering_link, origin xyz=0 0 0 rpy=0 0 0, axis 0.0 0.0 1.0, limit lower=-0.6981 upper=0.6981 effort=100 velocity=3.0
- joint front_left_wheel_joint: origin xyz=0.25 0.15 -0.05 rpy=1.57 0 0 -> xyz=0.25 0.15 -0.05 rpy=1.57 0.0 0.0; parent base_link -> wheel_steering_link
- joint front_right_wheel_joint: origin xyz=0.25 -0.15 -0.05 rpy=1.57 0 0 -> xyz=0.25 -0.15 -0.05 rpy=1.57 0.0 0.0; parent base_link -> wheel_steering_link
- joint rear_left_wheel_joint: origin xyz=-0.25 0.15 -0.05 rpy=1.57 0 0 -> xyz=-0.25 0.15 -0.05 rpy=1.57 0.0 0.0
- joint rear_right_wheel_joint: origin xyz=-0.25 -0.15 -0.05 rpy=1.57 0 0 -> xyz=-0.25 -0.15 -0.05 rpy=1.57 0.0 0.0
