Commit message: Added RemoteUI.py teleop program

File: urdf/messibotcopy.urdf (robot description, URDF)
Before this commit: robot messi_bot, 8 links, 7 joints
Links:
- link front_caster_of_wheel: mass 0.1 -> 0.05
- link front_wheel: mass 0.1 -> 0.05
- link left_finger: mass 0.1 -> 0.01
- link left_wheel: mass 0.01 -> 0.05
- link right_wheel: mass 0.1 -> 0.05
